Commit message: renaming to IsaacLab convetion; Hide all taxel links

File: urdf/4x4n.xacro (robot description, xacro)
@@ -18,5 +18,5 @@
         <origin xyz="0 0 0" rpy="0 0 0" />
         <geometry>
-          <mesh filename="package://official_xela_models/mesh/4x4.stl"/>
+          <mesh filename="package://official_xela_models/mesh/sensor_4x4.stl"/>
         </geometry>
       </collision>
@@ -25,5 +25,5 @@
           <origin xyz="0 0 0" rpy="0 0 0" />
           <geometry>
-            <mesh filename="package://official_xela_models/mesh/4x4.stl"/>
+            <mesh filename="package://official_xela_models/mesh/sensor_4x4.stl"/>
           </geometry>
           <material name="${col}"/>

File: urdf/allegro_hand_right_curved.xacro (robot description, xacro)
@@ -4,5 +4,7 @@
 	<xacro:include filename="$(find official_xela_models)/urdf/allegro_hand_right_new.xacro" />
 	<link name="world" />
+	<!-- <xacro:allegro_hand_right_new sequence="0" tips="curved" parent="world"  -->
+								  <!-- defaultnames="1" palm="1" taxels="1" /> -->
 	<xacro:allegro_hand_right_new sequence="0" tips="curved" parent="world"
-								  defaultnames="1" palm="1" taxels="1" />
+								  defaultnames="1" palm="1" taxels="0" />
 </robot>

File: urdf/allegro_hand_right_new.xacro (robot description, xacro)
@@ -213,5 +213,5 @@
         <visual>
           <geometry>
-            <mesh filename="package://official_xela_models/mesh/allegro/link_0.0_ext.STL" />
+            <mesh filename="package://official_xela_models/mesh/allegro/link_0_ext.STL" />
           </geometry>
           <material name="grey"/>
@@ -229,5 +229,5 @@
         </inertial>
       </link>
-      <joint name="joint_${finger_num*4+0}.0" type="revolute">
+      <joint name="joint_${finger_num*4+0}" type="revolute">
         <axis xyz="0 0 1"/>
         <limit effort="15" velocity="7" lower="${-0.57+0.1}" upper="${0.57-0.1}" />
@@ -240,5 +240,5 @@
           <geometry>
             <xacro:if value="${phalanges == 1}">
-              <mesh filename="package://official_xela_models/mesh/allegro/link_1.0.stl" />
+              <mesh filename="package://official_xela_models/mesh/allegro/link_1.stl" />
             </xacro:if>
             <xacro:if value="${phalanges != 1}">
@@ -307,5 +307,5 @@
         <xacro:sensor4x4n x_seq="${x_seq}${finger_num*4+0}" col="red" parent="${sequence}link_${finger_num*4+1}" ry="90" z="0.021" y="-0.012" x="0.0108" body="1" taxels="${taxels}" skipinertia="1" />
       </xacro:if>
-      <joint name="joint_${finger_num*4+1}.0" type="revolute">
+      <joint name="joint_${finger_num*4+1}" type="revolute">
         <limit effort="15" velocity="7" lower="${-0.296+0.1}" upper="${1.71-0.1}" />
         <axis xyz="0 1 0"/>
@@ -318,5 +318,5 @@
           <geometry>
             <xacro:if value="${phalanges == 1}">
-              <mesh filename="package://official_xela_models/mesh/allegro/link_2.0.stl" />
+              <mesh filename="package://official_xela_models/mesh/allegro/link_2.stl" />
             </xacro:if>
             <xacro:if value="${phalanges != 1}">
@@ -381,5 +381,5 @@
         <xacro:sensor4x4n x_seq="${x_seq}${finger_num*4+2}" col="red" parent="${sequence}link_${finger_num*4+2}" ry="90" z="0.0445" y="-0.012" x="0.01" body="1" taxels="${taxels}" skipinertia="1" />
       </xacro:if>
-      <joint name="joint_${finger_num*4+2}.0" type="revolute">
+      <joint name="joint_${finger_num*4+2}" type="revolute">
         <axis xyz="0 1 0"/>
         <limit effort="15" velocity="7" lower="${-0.274+0.1}" upper="${1.809-0.1}" />
@@ -391,5 +391,5 @@
         <visual>
           <geometry>
-            <mesh filename="package://official_xela_models/mesh/allegro/link_3.0.STL" />
+            <mesh filename="package://official_xela_models/mesh/allegro/link_3.STL" />
           </geometry>
           <material name="black" />
@@ -423,5 +423,5 @@
         </xacro:unless>
       </link>
-      <joint name="joint_${finger_num*4+3}.0" type="revolute">
+      <joint name="joint_${finger_num*4+3}" type="revolute">
         <axis xyz="0 1 0"/>
         <limit effort="15" velocity="7" lower="${-0.327+0.1}" upper="${1.718-0.1}" />
@@ -447,5 +447,5 @@
         <visual>
           <geometry>
-            <mesh filename="package://official_xela_models/mesh/allegro/link_12.0_right.STL" />
+            <mesh filename="package://official_xela_models/mesh/allegro/link_12_right.STL" />
           </geometry>
           <material name="grey" />
@@ -463,5 +463,5 @@
         </inertial>
       </link>
-      <joint name="joint_${finger_num*4+0}.0" type="revolute">
+      <joint name="joint_${finger_num*4+0}" type="revolute">
         <axis xyz="-1 0 0"/>
         <limit effort="15" velocity="7" lower="${0.363-0.1}" upper="${1.496-0.1}" />
@@ -473,5 +473,5 @@
         <visual>
           <geometry>
-            <mesh filename="package://official_xela_models/mesh/allegro/link_13.0.STL" />
+            <mesh filename="package://official_xela_models/mesh/allegro/link_13.STL" />
           </geometry>
           <material name="grey" />
@@ -510,5 +510,5 @@
         </joint>
       </xacro:if>
-      <joint name="joint_${finger_num*4+1}.0" type="revolute">
+      <joint name="joint_${finger_num*4+1}" type="revolute">
         <axis xyz="0 0 1"/>
         <limit effort="15" velocity="7" lower="${-0.205+0.1}" upper="${1.263-0.1}" />
@@ -521,5 +521,5 @@
           <geometry>
             <xacro:if value="${phalanges == 1}">
-              <mesh filename="package://official_xela_models/mesh/allegro/thumb_1.0.stl"/>
+              <mesh filename="package://official_xela_models/mesh/allegro/thumb_1.stl"/>
             </xacro:if>
             <xacro:if value="${phalanges != 1}">
@@ -583,5 +583,5 @@
         <xacro:sensor4x4n x_seq="${x_seq}${finger_num*4+1}" parent="${sequence}link_${finger_num*4+2}" ry="90" z="0.023" y="-0.012" x="0.011" body="1" taxels="${taxels}" skipinertia="1" />
       </xacro:if>
-      <joint name="joint_${finger_num*4+2}.0" type="revolute">
+      <joint name="joint_${finger_num*4+2}" type="revolute">
         <axis xyz="0 1 0"/>
         <limit effort="15" velocity="7" lower="${-0.289+0.1}" upper="${1.744-0.1}" />
@@ -594,5 +594,5 @@
           <geometry>
             <xacro:if value="${phalanges == 1}">
-              <mesh filename="package://official_xela_models/mesh/allegro/thumb_2.0.stl"/>
+              <mesh filename="package://official_xela_models/mesh/allegro/thumb_2.stl"/>
             </xacro:if>
             <xacro:if value="${phalanges != 1}">
@@ -683,5 +683,5 @@
         <xacro:sensor4x4n x_seq="${x_seq}${finger_num*4+2}" parent="${sequence}link_${finger_num*4+3}" ry="90" z="0.021" y="-0.012" x="0.011" body="1" taxels="${taxels}" skipinertia="1" />
       </xacro:if>
-    <joint name="joint_${finger_num*4+3}.0" type="revolute">
+    <joint name="joint_${finger_num*4+3}" type="revolute">
       <axis xyz="0 1 0"/>
       <limit effort="15" velocity="7" lower="${-0.262+0.1}" upper="${1.819-0.1}" />

File: urdf/taxel_n.xacro (robot description, xacro)
@@ -5,10 +5,10 @@
   <!-- <xacro:taxel_n sequence="${sequence}_4x6_01" x="${1*txstep+xoff}" y="${4*tystep-yoff}" z="${zoff}" parent="${bseq}_4x6_link" sensor_collision="${sensor_collision}" /> -->
   <xacro:macro name="taxel_n" params="sequence parent x:=0.0 y:=0.0 z:=0.0 rx:=0.0 ry:=0.0 rz:=0.0 col:='blue' zmod:=0.0 sensor_collision:=1 sensor_inertial:=0">
-    <joint name="${sequence}_joint" type="prismatic">
+    <joint name="${sequence}_joint" type="fixed">
       <origin xyz="${x} ${y} ${z}" rpy="${radians(rx)} ${radians(ry)} ${radians(rz)}"/>
       <parent link="${parent}"/>
       <child link="${sequence}_link"/>
       <axis xyz="0 0 1"/>
-      <limit effort="100.0" lower="${-0.001-zmod}" upper="0.000" velocity="0.5"/>
+      <!-- <limit effort="100.0" lower="${-0.001-zmod}" upper="0.000" velocity="0.5"/> -->
     </joint>
     <link name="${sequence}_link">
